Commit message: adding updates

File: honeybee_description/urdf/honeybee_description.urdf.xacro (robot description, xacro)
@@ -1,22 +1,46 @@
 <?xml version="1.0"?>
-<robot xmlns:xacro="http://ros.org/wiki/xacro">
-  <!-- Description Package -->
-  <xacro:property name="package"      value="ona01_description" />
+<robot xmlns:xacro="http://www.ros.org/wiki/xacro" name="honeybee">
+  <!-- Properties -->
+  <xacro:property name="package"      value="honeybee_description" />
   <xacro:property name="find_package" value="$(find ${package})" />
+  <xacro:property name="meshes"             value="${package}/meshes/" />
+  <xacro:property name="realsense_mount"    value="realsense_fixed_mount.STL" />
   <!-- Includes -->
   <xacro:include filename="${find_package}/urdf/includes/custom_macros.urdf.xacro" />
   <xacro:include filename="${find_package}/urdf/includes/OS0-32.urdf.xacro" />
-  <!-- MESHES -->
-  <xacro:property name="meshes"             value="${package}/meshes/" />
-  <xacro:property name="realsense_mount"    value="realsense_fixed_mount.STL" />
-  <!-- ARK Bulkhead Top Ref. Link -->
+  <xacro:include filename="$(find clearpath_platform_description)/urdf/common.urdf.xacro"/>
+  <xacro:include filename="$(find clearpath_platform_description)/urdf/j100/j100.urdf.xacro"/>
+  <xacro:include filename="$(find clearpath_platform_description)/urdf/j100/attachments/fender.urdf.xacro"/>
+  <xacro:include filename="$(find clearpath_platform_description)/urdf/j100/attachments/top_plate.urdf.xacro"/>
+  <xacro:include filename="$(find clearpath_sensors_description)/urdf/intel_realsense.urdf.xacro"/>
+  <xacro:include filename="$(find clearpath_sensors_description)/urdf/microstrain_imu.urdf.xacro"/>
+  <!-- Clearpath base platform -->
+  <xacro:j100 wheel="default"/>
+  <xacro:fender name="front_fender" model="default" parent_link="base_link">
+    <origin xyz="0.0 0.0 0.0" rpy="0.0 0.0 0.0"/>
+  </xacro:fender>
+  <xacro:fender name="rear_fender" model="default" parent_link="base_link">
+    <origin xyz="0.0 0.0 0.0" rpy="0.0 0.0 3.1415"/>
+  </xacro:fender>
+  <xacro:top_plate name="ark_enclosure" model="ark_enclosure" parent_link="default_mount">
+    <origin xyz="0.0 0.0 0.0" rpy="0.0 0.0 0.0"/>
+  </xacro:top_plate>
+  <!-- Metal enclosure -->
   <xacro:link name="ark_enclosure_top" parent="ark_enclosure_link" type="fixed">
   	<origin xyz="0 0 0.06803" rpy="0 0 0" />
   </xacro:link>
-  <!-- RealSense Mount -->
+  <!-- Sensors -->
+  <xacro:intel_realsense name="camera_0" parent_link="realsense_mount_link" update_rate="30" image_height="480" image_width="640">
+    <origin xyz="0.0 0.0 0.004" rpy="0.0 0.0 0.0"/>
+  </xacro:intel_realsense>
   <xacro:mesh name="realsense_mount" parent="ark_enclosure_top_link" mesh="${realsense_mount}" material="cpr_grey">
     <origin xyz="0.1344 0 0" rpy="0 0 0" />
   </xacro:mesh>
-  <!-- Ouster Tower -->
+  <xacro:microstrain_imu name="imu_1" parent_link="base_link" update_rate="100">
+    <origin xyz="0.093 0.103 0.1881" rpy="0.0 0.0 -1.57"/>
+  </xacro:microstrain_imu>
+  <xacro:OS0-32 parent="ouster_tower_mount_plate">
+    <origin xyz="0 0 0" rpy="0 0 0" />
+  </xacro:OS0-32>
   <xacro:mount_plate prefix="ouster_tower" parent="ark_enclosure_top_link" pattern=".08 .08" height="0.125" radius="0.005">
     <xacro:property name="plate"     value="0 0 0" />
@@ -24,7 +48,3 @@
     <xacro:property name="rpy"       value="0 0 0" />
   </xacro:mount_plate>
-  <!-- Ouster Lidar -->
-  <xacro:OS0-32 parent="ouster_tower_mount_plate">
-    <origin xyz="0 0 0" rpy="0 0 0" />
-  </xacro:OS0-32>
 </robot>

File: honeybee_description/urdf/includes/OS0-32.urdf.xacro (robot description, xacro)
@@ -50,5 +50,5 @@
          <origin xyz="0 0 0.0" rpy="0 0 1.5707" />
          <geometry>
-	         <mesh filename="package://ona01_description/meshes/os1_64.dae" />
+	         <mesh filename="package://honeybee_description/meshes/os1_64.dae" />
            <!-- <cylinder length="0.073" radius="0.04" /> -->
          </geometry>

Commit message: sensor sim

File: honeybee_description/urdf/honeybee_description.urdf.xacro (robot description, xacro)
@@ -9,10 +9,10 @@
   <xacro:include filename="${find_package}/urdf/includes/custom_macros.urdf.xacro" />
   <xacro:include filename="${find_package}/urdf/includes/OS0-32.urdf.xacro" />
+  <xacro:include filename="${find_package}/urdf/includes/intel_realsense.urdf.xacro"/>
+  <xacro:include filename="${find_package}/urdf/includes/microstrain_imu.urdf.xacro"/>
+  <xacro:include filename="${find_package}/urdf/includes/j100.urdf.xacro"/>
   <xacro:include filename="$(find clearpath_platform_description)/urdf/common.urdf.xacro"/>
-  <xacro:include filename="$(find clearpath_platform_description)/urdf/j100/j100.urdf.xacro"/>
   <xacro:include filename="$(find clearpath_platform_description)/urdf/j100/attachments/fender.urdf.xacro"/>
   <xacro:include filename="$(find clearpath_platform_description)/urdf/j100/attachments/top_plate.urdf.xacro"/>
-  <xacro:include filename="$(find clearpath_sensors_description)/urdf/intel_realsense.urdf.xacro"/>
-  <xacro:include filename="$(find clearpath_sensors_description)/urdf/microstrain_imu.urdf.xacro"/>
   <!-- Clearpath base platform -->
   <xacro:j100 wheel="default"/>
@@ -40,6 +40,6 @@
     <origin xyz="0.093 0.103 0.1881" rpy="0.0 0.0 -1.57"/>
   </xacro:microstrain_imu>
-  <xacro:OS0-32 parent="ouster_tower_mount_plate">
-    <origin xyz="0 0 0" rpy="0 0 0" />
+  <xacro:OS0-32 parent="ouster_tower_custom_mount"> <!-- Steve mod: for some rason _mount_plate didn't work, so removed -->
+    <origin xyz="0 0 0.125" rpy="0 0 0" />
   </xacro:OS0-32>
   <xacro:mount_plate prefix="ouster_tower" parent="ark_enclosure_top_link" pattern=".08 .08" height="0.125" radius="0.005">

File: honeybee_description/urdf/includes/OS0-32.urdf.xacro (robot description, xacro)
@@ -51,5 +51,4 @@
          <geometry>
 	         <mesh filename="package://honeybee_description/meshes/os1_64.dae" />
-           <!-- <cylinder length="0.073" radius="0.04" /> -->
          </geometry>
       </visual>
@@ -69,55 +68,39 @@
       <origin xyz="0.0 0.0 0.03618" rpy="0 0 0" />
     </joint>
-    <!-- Gazebo requires the ouster_gazebo_plugins package -->
     <gazebo reference="${name}">
-        <sensor type="ray" name="${name}-OS0-32">
-          <pose>0 0 0 0 0 0</pose>
-          <visualize>false</visualize>
-          <update_rate>${hz}</update_rate>
-          <ray>
-            <scan>
-              <horizontal>
-                <samples>${samples}</samples>
-                <resolution>1</resolution>
-                <min_angle>${min_angle}</min_angle>
-                <max_angle>${max_angle}</max_angle>
-              </horizontal>
-              <vertical>
-                <samples>${lasers}</samples>
-                <resolution>1</resolution>
-                <min_angle>${vfov_min}</min_angle>
-                <max_angle>${vfov_max}</max_angle>
-              </vertical>
-            </scan>
-            <range>
-              <min>${min_range}</min>
-              <max>${max_range}</max>
-              <resolution>0.03</resolution>
-            </range>
-          </ray>
-          <plugin name="gazebo_ros_laser_controller" filename="libgazebo_ros_ouster_laser.so">
-            <topicName>${topic_points}</topicName>
-            <frameName>${lidar_link}</frameName>
-            <min_range>${min_range}</min_range>
-            <max_range>${max_range}</max_range>
-            <gaussianNoise>${noise}</gaussianNoise>
-          </plugin>
-        </sensor>
+      <sensor name="${name}" type="gpu_lidar">
+        <update_rate>${hz}</update_rate>
+        <visualize>false</visualize>
+        <always_on>true</always_on>
+        <ignition_frame_id>${name}</ignition_frame_id>  <!-- Steve mod: fix frame to something actually in URDF -->
+        <topic>sensors/lidar_0</topic>  <!-- Steve mod: set topic to same as hardware -->
+        <lidar>
+          <scan>
+            <horizontal>
+              <samples>${samples}</samples>
+              <resolution>1</resolution>
+              <min_angle>${min_angle}</min_angle>
+              <max_angle>${max_angle}</max_angle>
+            </horizontal>
+            <vertical>
+              <samples>${lasers}</samples>
+              <resolution>1</resolution>
+              <min_angle>${vfov_min}</min_angle>
+              <max_angle>${vfov_max}</max_angle>
+            </vertical>
+          </scan>
+          <range>
+            <min>${min_range}</min>
+            <max>${max_range}</max>
+            <resolution>0.003</resolution>
+          </range>
+          <noise>
+            <type>gaussian</type>
+            <mean>0.0</mean>
+            <stddev>0.003</stddev>
+          </noise>
+        </lidar>
+      </sensor>
     </gazebo>
-    <!-- IMU -->
-  <gazebo>
-    <plugin name="imu_controller" filename="libhector_gazebo_ros_imu.so">
-      <robotNamespace>/</robotNamespace>
-      <updateRate>100.0</updateRate>
-      <bodyName>${imu_link}</bodyName>
-      <topicName>${topic_imu}</topicName>
-      <accelDrift>0.005 0.005 0.005</accelDrift>
-      <accelGaussianNoise>0.005 0.005 0.005</accelGaussianNoise>
-      <rateDrift>0.005 0.005 0.005 </rateDrift>
-      <rateGaussianNoise>0.005 0.005 0.005 </rateGaussianNoise>
-      <headingDrift>0.005</headingDrift>
-      <headingGaussianNoise>0.005</headingGaussianNoise>
-    </plugin>
-  </gazebo>
   </xacro:macro>
 </robot>

File: honeybee_description/urdf/includes/mount_plate.urdf.xacro (robot description, xacro)
@@ -20,5 +20,6 @@
     #####################################################-->
     <link name="${prefix}_custom_mount" />
-    <link name="${prefix}_mount_plate">
+    <!-- Steve: for some rason _mount_plate crashes with dart errors, so removed -->
+    <!-- <link name="${prefix}_mount_plate">
       <visual>
         <material name="cpr_grey" />
@@ -34,5 +35,5 @@
         <origin xyz="0 0 -${(plate_height/2)}" rpy="0 0 0" />
       </collision>
-    </link>
+    </link> -->
     <joint name="${prefix}_custom_mount_joint" type="fixed">
       <parent link="${parent}" />
@@ -41,9 +42,9 @@
       <!--<xacro:insert_block name="origin" />-->
     </joint>
-    <joint name="${prefix}_mount_plate_joint" type="fixed">
+    <!-- <joint name="${prefix}_mount_plate_joint" type="fixed">
       <parent link="${prefix}_custom_mount" />
       <child link="${prefix}_mount_plate" />
       <origin xyz="0 0 ${(height+plate_height)}" rpy="0 0 0" />
-    </joint>
+    </joint> -->
     <!--#################################################
                           LEG LINKS
@@ -139,19 +140,3 @@
     </xacro:if>
   </xacro:macro>
-  <xacro:if value="$(optenv MOUNT_PLATE_ENABLED 0)">
-    <xacro:property name="prefix"                    value="$(optenv MOUNT_PLATE_PREFIX tower)" />
-    <xacro:property name="parent"                    value="$(optenv MOUNT_PLATE_PARENT base_link)" />
-    <xacro:property name="height"                    value="$(optenv MOUNT_TOWER_HEIGHT 0)" />
-    <xacro:property name="radius"                    value="$(optenv MOUNT_LEG_RADIUS 0.003)" />
-    <xacro:property name="dimensions"                value="$(optenv MOUNT_PLATE_DIMENSIONS 0.140 0.140 0.00635)" />
-    <xacro:property name="pattern"                   value="$(optenv MOUNT_PLATE_PATTERN 0 0)" />
-    <xacro:property name="xyz"                       value="$(optenv MOUNT_PLATE_XYZ 0 0 0)" />
-    <xacro:property name="rpy"                       value="$(optenv MOUNT_PLATE_RPY 0 0 0)" />
-    <xacro:mount_plate prefix="${prefix}" parent="${parent}" height="${height}" pattern="${pattern}" radius="${radius}">
-      <xacro:property name="plate"     value="${dimensions}" lazy_eval="false" />
-      <xacro:property name="radius"    value="${radius}"     lazy_eval="false" />
-      <xacro:property name="xyz"       value="${xyz}"        lazy_eval="false" />
-      <xacro:property name="rpy"       value="${rpy}"        lazy_eval="false" />
-    </xacro:mount_plate>
-  </xacro:if>
 </robot>

Commit message: fix frame flip

File: honeybee_description/urdf/honeybee_description.urdf.xacro (robot description, xacro)
@@ -6,4 +6,5 @@
   <xacro:property name="meshes"             value="${package}/meshes/" />
   <xacro:property name="realsense_mount"    value="realsense_fixed_mount.STL" />
+  <xacro:arg      name="is_sim"       default="false"/>
   <!-- Includes -->
   <xacro:include filename="${find_package}/urdf/includes/custom_macros.urdf.xacro" />
@@ -40,5 +41,5 @@
     <origin xyz="0.093 0.103 0.1881" rpy="0.0 0.0 -1.57"/>
   </xacro:microstrain_imu>
-  <xacro:OS0-32 parent="ouster_tower_custom_mount"> <!-- Steve mod: for some rason _mount_plate didn't work, so removed -->
+  <xacro:OS0-32 parent="ouster_tower_custom_mount" is_sim="$(arg is_sim)"> <!-- Steve mod: for some rason _mount_plate didn't work, so removed -->
     <origin xyz="0 0 0.125" rpy="0 0 0" />
   </xacro:OS0-32>

File: honeybee_description/urdf/includes/OS0-32.urdf.xacro (robot description, xacro)
@@ -2,5 +2,5 @@
 <robot xmlns:xacro="http://www.ros.org/wiki/xacro" name="OS0-32">
   <xacro:property name="M_PI" value="3.1415926535897931" />
-  <xacro:macro name="OS0-32" params="*origin parent:=base_link name:=os0_sensor topic_points:=/os0_cloud_node/points topic_imu:=/os0_cloud_node/imu hz:=10 lasers:=32 samples:=512 min_range:=0.9 max_range:=75.0 noise:=0.008 min_angle:=-${M_PI} max_angle:=${M_PI} lidar_link:=os0_lidar imu_link:=os0_imu vfov_min:=-0.785398 vfov_max:=0.785398">
+  <xacro:macro name="OS0-32" params="*origin parent:=base_link name:=os0_sensor topic_points:=/os0_cloud_node/points topic_imu:=/os0_cloud_node/imu hz:=10 lasers:=32 samples:=512 min_range:=0.9 max_range:=75.0 noise:=0.008 min_angle:=-${M_PI} max_angle:=${M_PI} lidar_link:=os0_lidar imu_link:=os0_imu vfov_min:=-0.785398 vfov_max:=0.785398 is_sim:=false">
     <joint name="${name}_mount_joint" type="fixed">
       <xacro:insert_block name="origin" />
@@ -54,18 +54,21 @@
       </visual>
     </link>
-    <link name="${imu_link}" />
-    <link name="${lidar_link}" />
-    <joint name="${name}_imu_link_joint" type="fixed">
-      <parent link="${name}" />
-      <child link="${imu_link}" />
-      <origin xyz="0.006253 -0.011775 0.007645" rpy="0 0 0" />
-    </joint>
-    <gazebo reference="${imu_link}">
-    </gazebo>
-    <joint name="${name}_lidar_link_joint" type="fixed">
-      <parent link="${name}" />
-      <child link="${lidar_link}" />
-      <origin xyz="0.0 0.0 0.03618" rpy="0 0 0" />
-    </joint>
+    <!-- Steve mod: cannot use on hardware since it publishes its own frames -->
+    <xacro:if value="${is_sim}">
+      <link name="${imu_link}" />
+      <link name="${lidar_link}" />
+      <joint name="${name}_imu_link_joint" type="fixed">
+        <parent link="${name}" />
+        <child link="${imu_link}" />
+        <origin xyz="0.006253 -0.011775 0.007645" rpy="0 0 0" />
+      </joint>
+      <gazebo reference="${imu_link}">
+      </gazebo>
+      <joint name="${name}_lidar_link_joint" type="fixed">
+        <parent link="${name}" />
+        <child link="${lidar_link}" />
+        <origin xyz="0.0 0.0 0.03618" rpy="0 0 0" />
+      </joint>
+    </xacro:if>
     <gazebo reference="${name}">
       <sensor name="${name}" type="gpu_lidar">

Commit message: Now passing correct control parameter
Signed-off-by: Abhishekh Reddy <helloarm@pm.me>

File: honeybee_description/urdf/honeybee_description.urdf.xacro (robot description, xacro)
@@ -18,5 +18,9 @@
   <!-- Clearpath base platform -->
   <!-- <xacro:j100 wheel="default"/> -->
+<<<<<<< Updated upstream
   <xacro:j100 control="diff_fwd" front_wheels="outdoor" rear_wheels="outdoor"/>
+=======
+  <xacro:j100 control="diff_4wd" front_wheels="outdoor" rear_wheels="outdoor"/>
+>>>>>>> Stashed changes
   <xacro:fender name="front_fender" model="default" parent_link="base_link">
     <origin xyz="0.0 0.0 0.0" rpy="0.0 0.0 0.0"/>

File: honeybee_description/urdf/includes/j100.urdf.xacro (robot description, xacro)
@@ -17,5 +17,9 @@
   <xacro:property name="dummy_inertia" value="1e-09"/>
   <xacro:property name="mount_spacing" value="0.120" />
+<<<<<<< Updated upstream
   <xacro:macro name="j100" params="control:='diff_fwd' front_wheels:='outdoor' rear_wheels:='outdoor'">
+=======
+  <xacro:macro name="j100" params="control:='diff_4wd' front_wheels:='outdoor' rear_wheels:='outdoor'">
+>>>>>>> Stashed changes
     <link name="base_link"></link>
     <joint name="base_link_joint" type="fixed">
