Commit message: Resolved merge conflict
Signed-off-by: Abhishekh Reddy <helloarm@pm.me>

File: honeybee_description/urdf/includes/j100.urdf.xacro (robot description, xacro)
@@ -17,9 +17,5 @@
   <xacro:property name="dummy_inertia" value="1e-09"/>
   <xacro:property name="mount_spacing" value="0.120" />
-<<<<<<< Updated upstream
-  <xacro:macro name="j100" params="control:='diff_fwd' front_wheels:='outdoor' rear_wheels:='outdoor'">
-=======
   <xacro:macro name="j100" params="control:='diff_4wd' front_wheels:='outdoor' rear_wheels:='outdoor'">
->>>>>>> Stashed changes
     <link name="base_link"></link>
     <joint name="base_link_joint" type="fixed">
